Commit message: TEMP

File: dragon_description/urdf/dragon_three_dof.gazebo.xacro (robot description, xacro)
@@ -1,112 +1,7 @@
 <?xml version="1.0"?>
-<robot xmlns:xacro="http://www.ros.org/wiki/xacro" name="dragon">
-	<xacro:macro name="Links" params="Name Color">
-		<gazebo reference="${Name}">
-			<material>Gazebo/${Color}</material>
-			<kp>1000000.0</kp>
-			<kd>100.0</kd>
-			<mu1>1.5</mu1>
-			<mu2>1.5</mu2>
-			<fdir1>0 1 0</fdir1>
-			<maxVel>1.0</maxVel>
-			<minDepth>0.005</minDepth>
-			<selfCollide>true</selfCollide>
-			<static>false</static>
-			<turnGravityOff>false</turnGravityOff>
-		</gazebo>
-	</xacro:macro>
-	<xacro:macro name="Feet" params="Name">
-		<gazebo reference="${Name}">
-			<material>Gazebo/Yellow</material>
-			<mu1>1.5</mu1>
-			<mu2>1.5</mu2>
-			<fdir1>0 1 0</fdir1>
-			<maxVel>1.0</maxVel>
-			<minDepth>0.005</minDepth>
-			<selfCollide>true</selfCollide>
-			<static>false</static>
-			<turnGravityOff>false</turnGravityOff>
-		</gazebo>
-	</xacro:macro>
-	<xacro:Links Name="body"              Color="Green"/>
-	<xacro:Links Name="left_front_upper"  Color="Turquoise"/>
-	<xacro:Links Name="right_front_upper" Color="Turquoise"/>
-	<xacro:Links Name="left_back_upper"   Color="Turquoise"/>
-	<xacro:Links Name="right_back_upper"  Color="Turquoise"/>
-	<xacro:Links Name="left_front_leg"    Color="Blue"/>
-	<xacro:Links Name="right_front_leg"   Color="Blue"/>
-	<xacro:Links Name="left_back_leg"     Color="Blue"/>
-	<xacro:Links Name="right_back_leg"    Color="Blue"/>
-	<xacro:Links Name="left_front_shine"  Color="Red"/>
-	<xacro:Links Name="right_front_shine" Color="Red"/>
-	<xacro:Links Name="left_back_shine"   Color="Orange"/>
-	<xacro:Links Name="right_back_shine"  Color="Orange"/>
-	<xacro:Feet Name="left_front_feet"  />
-	<xacro:Feet Name="right_front_feet" />
-	<xacro:Feet Name="left_back_feet"   />
-	<xacro:Feet Name="right_back_feet"  />
+<robot xmlns:xacro="http://www.ros.org/wiki/xacro" name="dragon_gazebo">
 	<!-- ROS-Control plugin -->
 	<gazebo>
-		<plugin name="ros_control" filename="libgazebo_ros_control.so">
-	</gazebo>
-	<!-- IMU plugin -->
-	<gazebo>
-		<plugin name="imu_plugin" filename="libgazebo_ros_imu.so">
-			<alwaysOn>true</alwaysOn>
-			<bodyName>body</bodyName>
-			<topicName>/dragon/imu</topicName>
-			<serviceName>/dragon/imu_service</serviceName>
-			<gaussianNoise>0.0</gaussianNoise>
-			<updateRate>20.0</updateRate>
-		</plugin>
-	</gazebo>
-	<!-- Contact Force plugin -->
-	<gazebo reference="left_front_feet">
-		<sensor name="lf_contact_sensor" type="contact">
-			<always_on>true</always_on>
-			<update_rate>30.0</update_rate>
-			<contact>
-				<collision>left_front_feet_collision</collision>
-			</contact>
-			<plugin name="lf_foot_bumper" filename="libgazebo_ros_bumper.so">
-				<bumperTopicName>/dragon/lf_contact_sensor_state</bumperTopicName>
-			</plugin>
-		</sensor>
-	</gazebo>
-	<gazebo reference="right_front_feet">
-		<sensor name="rf_contact_sensor" type="contact">
-			<always_on>true</always_on>
-			<update_rate>30.0</update_rate>
-			<contact>
-				<collision>right_front_feet_collision</collision>
-			</contact>
-			<plugin name="rf_foot_bumper" filename="libgazebo_ros_bumper.so">
-				<bumperTopicName>/dragon/rf_contact_sensor_state</bumperTopicName>
-			</plugin>
-		</sensor>
-	</gazebo>
-	<gazebo reference="left_back_feet">
-		<sensor name="lb_contact_sensor" type="contact">
-			<always_on>true</always_on>
-			<update_rate>30.0</update_rate>
-			<contact>
-				<collision>left_back_feet_collision</collision>
-			</contact>
-			<plugin name="lb_foot_bumper" filename="libgazebo_ros_bumper.so">
-				<bumperTopicName>/dragon/lb_contact_sensor_state</bumperTopicName>
-			</plugin>
-		</sensor>
-	</gazebo>
-	<gazebo reference="right_back_feet">
-		<sensor name="rb_contact_sensor" type="contact">
-			<always_on>true</always_on>
-			<update_rate>30.0</update_rate>
-			<contact>
-				<collision>right_back_feet_collision</collision>
-			</contact>
-			<plugin name="rb_foot_bumper" filename="libgazebo_ros_bumper.so">
-				<bumperTopicName>/dragon/rb_contact_sensor_state</bumperTopicName>
-			</plugin>
-		</sensor>
+		<plugin name="ros_control" filename="libgazebo_ros_control.so"/>
 	</gazebo>
 </robot>
