Commit message: this is debug version

File: qr_description/urdf/dinasour.transmission.xacro (robot description, xacro)
@@ -22,14 +22,14 @@
 		</transmission>
 	</xacro:macro>
-	<xacro:Trans Name="left_front_pitch" />
+	<xacro:Trans Name="left_front_yaw" />
 	<xacro:Trans Name="left_front_hip" />
 	<xacro:Trans Name="left_front_knee" />
-	<xacro:Trans Name="right_front_pitch" />
+	<xacro:Trans Name="right_front_yaw" />
 	<xacro:Trans Name="right_front_hip" />
 	<xacro:Trans Name="right_front_knee" />
-	<xacro:Trans Name="left_back_pitch" />
+	<xacro:Trans Name="left_back_yaw" />
 	<xacro:Trans Name="left_back_hip" />
 	<xacro:Trans Name="left_back_knee" />
-	<xacro:Trans Name="right_back_pitch" />
+	<xacro:Trans Name="right_back_yaw" />
 	<xacro:Trans Name="right_back_hip" />
 	<xacro:Trans Name="right_back_knee" />

File: qr_description/urdf/dinasour.urdf.xacro (robot description, xacro)
@@ -65,5 +65,5 @@
 			</inertial>
 		</link>
-		<joint name="${Name}_pitch" type="revolute">
+		<joint name="${Name}_yaw" type="revolute">
 			<origin xyz="${X_Dir*(BODY_X/2-SHOD_L/2)} ${Y_Dir*(BODY_Y/2-SHOD_R)} ${-SHOD_R*2}" rpy="0 0 0"/>
 			<parent link="${Parent_Link}"/>

File: qr_description/urdf/single_leg.gazebo.xacro (robot description, xacro)
@@ -7,7 +7,7 @@
  </xacro:macro>
 	<xacro:Links Name="body"                 Color="Green"/>
-	<xacro:Links Name="left_front_shoulder"  Color="Turquoise"/>
-	<xacro:Links Name="left_front_leg"       Color="Blue"/>
-	<xacro:Links Name="left_front_shine"     Color="Red"/>
+	<xacro:Links Name="right_front_shoulder"  Color="Turquoise"/>
+	<xacro:Links Name="right_front_leg"       Color="Blue"/>
+	<xacro:Links Name="right_front_shine"     Color="Red"/>
 	<!-- ROS-Control plugin -->
  <gazebo>

File: qr_description/urdf/single_leg.transmission.xacro (robot description, xacro)
@@ -22,6 +22,6 @@
 		</transmission>
 	</xacro:macro>
-	<xacro:Trans Name="left_front_pitch" />
-	<xacro:Trans Name="left_front_hip" />
-	<xacro:Trans Name="left_front_knee" />
+	<xacro:Trans Name="right_front_yaw" />
+	<xacro:Trans Name="right_front_hip" />
+	<xacro:Trans Name="right_front_knee" />
 </robot>

File: qr_description/urdf/single_leg.urdf.xacro (robot description, xacro)
@@ -65,5 +65,5 @@
 			</inertial>
 		</link>
-		<joint name="${Name}_pitch" type="revolute">
+		<joint name="${Name}_yaw" type="revolute">
 			<origin xyz="${X_Dir*(BODY_X/2-SHOD_L/2)} ${Y_Dir*(BODY_Y/2-SHOD_R)} ${-SHOD_R*2}" rpy="0 0 0"/>
 			<parent link="${Parent_Link}"/>
@@ -138,7 +138,7 @@
 	<!--***************************************************************-->
 	<xacro:Body Name="body" Mass="10"/>
-	<xacro:Shoulder Name="left_front"  Mass="1" Parent_Link="body" X_Dir = "1"  Y_Dir = "-1"/>
-	<xacro:LEG Name="left_front"   Mass="1" Limit_Up = "2" Limit_Low="0"/>
-	<xacro:SHINE Name="left_front"  Mass="1" Limit_Up = "0" Limit_Low="-2"/>
+	<xacro:Shoulder Name="right_front"  Mass="1" Parent_Link="body" X_Dir = "1"  Y_Dir = "-1"/>
+	<xacro:LEG Name="right_front"   Mass="1" Limit_Up = "2" Limit_Low="0"/>
+	<xacro:SHINE Name="right_front"  Mass="1" Limit_Up = "0" Limit_Low="-2"/>
 	<link name="world"/>
 	<joint name="base_fixed" type="fixed">

File: qr_description/urdf/single_leg.xacro (robot description, xacro)
@@ -1,6 +1,6 @@
 <?xml version="1.0"?>
 <robot xmlns:xacro="http://www.ros.org/wiki/xacro" name="dragon">
-  <xacro:include filename="$(find dragon_description)/urdf/single_leg.urdf.xacro"/>
-  <xacro:include filename="$(find dragon_description)/urdf/single_leg.transmission.xacro"/>
-  <xacro:include filename="$(find dragon_description)/urdf/single_leg.gazebo.xacro"/>
+  <xacro:include filename="$(find qr_description)/urdf/single_leg.urdf.xacro"/>
+  <xacro:include filename="$(find qr_description)/urdf/single_leg.transmission.xacro"/>
+  <xacro:include filename="$(find qr_description)/urdf/single_leg.gazebo.xacro"/>
 </robot>
