Commit message: fix init bug

File: qr_description/urdf/dinasour.urdf.xacro (robot description, xacro)
@@ -146,8 +146,8 @@
 	<xacro:LEG Name="left_back"     Mass="1" Limit_Up = "2" Limit_Low="-2"/>
 	<xacro:LEG Name="right_back"    Mass="1" Limit_Up = "2" Limit_Low="-2"/>
-	<xacro:SHINE Name="left_front"  Mass="1" Limit_Up = "2" Limit_Low="-2"/>
-	<xacro:SHINE Name="right_front" Mass="1" Limit_Up = "2" Limit_Low="-2"/>
-	<xacro:SHINE Name="left_back"   Mass="1" Limit_Up = "2" Limit_Low="-2"/>
-	<xacro:SHINE Name="right_back"  Mass="1" Limit_Up = "2" Limit_Low="-2"/>
+	<xacro:SHINE Name="left_front"  Mass="1" Limit_Up = "2" Limit_Low="-2" />
+	<xacro:SHINE Name="right_front" Mass="1" Limit_Up = "2" Limit_Low="-2" />
+	<xacro:SHINE Name="left_back"   Mass="1" Limit_Up = "2" Limit_Low="-2" />
+	<xacro:SHINE Name="right_back"  Mass="1" Limit_Up = "2" Limit_Low="-2" />
 	<link name="world"/>
 	<joint name="base_fixed" type="fixed">

File: qr_description/urdf/dragon_three_dof.gazebo.xacro (robot description, xacro)
@@ -1,7 +1,112 @@
 <?xml version="1.0"?>
-<robot xmlns:xacro="http://www.ros.org/wiki/xacro" name="dragon_gazebo">
+<robot xmlns:xacro="http://www.ros.org/wiki/xacro" name="dragon">
+	<xacro:macro name="Links" params="Name Color">
+		<gazebo reference="${Name}">
+			<material>Gazebo/${Color}</material>
+			<kp>1000000.0</kp>
+			<kd>100.0</kd>
+			<mu1>1.5</mu1>
+			<mu2>1.5</mu2>
+			<fdir1>0 1 0</fdir1>
+			<maxVel>1.0</maxVel>
+			<minDepth>0.005</minDepth>
+			<selfCollide>true</selfCollide>
+			<static>false</static>
+			<turnGravityOff>false</turnGravityOff>
+		</gazebo>
+	</xacro:macro>
+	<xacro:macro name="Feet" params="Name">
+		<gazebo reference="${Name}">
+			<material>Gazebo/Yellow</material>
+			<mu1>1.5</mu1>
+			<mu2>1.5</mu2>
+			<fdir1>0 1 0</fdir1>
+			<maxVel>1.0</maxVel>
+			<minDepth>0.005</minDepth>
+			<selfCollide>true</selfCollide>
+			<static>false</static>
+			<turnGravityOff>false</turnGravityOff>
+		</gazebo>
+	</xacro:macro>
+	<xacro:Links Name="body"              Color="Green"/>
+	<xacro:Links Name="left_front_upper"  Color="Turquoise"/>
+	<xacro:Links Name="right_front_upper" Color="Turquoise"/>
+	<xacro:Links Name="left_back_upper"   Color="Turquoise"/>
+	<xacro:Links Name="right_back_upper"  Color="Turquoise"/>
+	<xacro:Links Name="left_front_leg"    Color="Blue"/>
+	<xacro:Links Name="right_front_leg"   Color="Blue"/>
+	<xacro:Links Name="left_back_leg"     Color="Blue"/>
+	<xacro:Links Name="right_back_leg"    Color="Blue"/>
+	<xacro:Links Name="left_front_shine"  Color="Red"/>
+	<xacro:Links Name="right_front_shine" Color="Red"/>
+	<xacro:Links Name="left_back_shine"   Color="Orange"/>
+	<xacro:Links Name="right_back_shine"  Color="Orange"/>
+	<xacro:Feet Name="left_front_feet"  />
+	<xacro:Feet Name="right_front_feet" />
+	<xacro:Feet Name="left_back_feet"   />
+	<xacro:Feet Name="right_back_feet"  />
 	<!-- ROS-Control plugin -->
 	<gazebo>
-		<plugin name="ros_control" filename="libgazebo_ros_control.so"/>
+		<plugin name="ros_control" filename="libgazebo_ros_control.so">
+	</gazebo>
+	<!-- IMU plugin -->
+	<gazebo>
+		<plugin name="imu_plugin" filename="libgazebo_ros_imu.so">
+			<alwaysOn>true</alwaysOn>
+			<bodyName>body</bodyName>
+			<topicName>/dragon/imu</topicName>
+			<serviceName>/dragon/imu_service</serviceName>
+			<gaussianNoise>0.0</gaussianNoise>
+			<updateRate>20.0</updateRate>
+		</plugin>
+	</gazebo>
+	<!-- Contact Force plugin -->
+	<gazebo reference="left_front_feet">
+		<sensor name="lf_contact_sensor" type="contact">
+			<always_on>true</always_on>
+			<update_rate>30.0</update_rate>
+			<contact>
+				<collision>left_front_feet_collision</collision>
+			</contact>
+			<plugin name="lf_foot_bumper" filename="libgazebo_ros_bumper.so">
+				<bumperTopicName>/dragon/lf_contact_sensor_state</bumperTopicName>
+			</plugin>
+		</sensor>
+	</gazebo>
+	<gazebo reference="right_front_feet">
+		<sensor name="rf_contact_sensor" type="contact">
+			<always_on>true</always_on>
+			<update_rate>30.0</update_rate>
+			<contact>
+				<collision>right_front_feet_collision</collision>
+			</contact>
+			<plugin name="rf_foot_bumper" filename="libgazebo_ros_bumper.so">
+				<bumperTopicName>/dragon/rf_contact_sensor_state</bumperTopicName>
+			</plugin>
+		</sensor>
+	</gazebo>
+	<gazebo reference="left_back_feet">
+		<sensor name="lb_contact_sensor" type="contact">
+			<always_on>true</always_on>
+			<update_rate>30.0</update_rate>
+			<contact>
+				<collision>left_back_feet_collision</collision>
+			</contact>
+			<plugin name="lb_foot_bumper" filename="libgazebo_ros_bumper.so">
+				<bumperTopicName>/dragon/lb_contact_sensor_state</bumperTopicName>
+			</plugin>
+		</sensor>
+	</gazebo>
+	<gazebo reference="right_back_feet">
+		<sensor name="rb_contact_sensor" type="contact">
+			<always_on>true</always_on>
+			<update_rate>30.0</update_rate>
+			<contact>
+				<collision>right_back_feet_collision</collision>
+			</contact>
+			<plugin name="rb_foot_bumper" filename="libgazebo_ros_bumper.so">
+				<bumperTopicName>/dragon/rb_contact_sensor_state</bumperTopicName>
+			</plugin>
+		</sensor>
 	</gazebo>
 </robot>

File: qr_description/urdf/single_leg.gazebo.xacro (robot description, xacro)
@@ -7,7 +7,7 @@
  </xacro:macro>
 	<xacro:Links Name="body"                 Color="Green"/>
-	<xacro:Links Name="right_front_shoulder"  Color="Turquoise"/>
-	<xacro:Links Name="right_front_leg"       Color="Blue"/>
-	<xacro:Links Name="right_front_shine"     Color="Red"/>
+	<xacro:Links Name="left_front_shoulder"  Color="Turquoise"/>
+	<xacro:Links Name="left_front_leg"       Color="Blue"/>
+	<xacro:Links Name="left_front_shine"     Color="Red"/>
 	<!-- ROS-Control plugin -->
  <gazebo>

File: qr_description/urdf/single_leg.transmission.xacro (robot description, xacro)
@@ -22,6 +22,6 @@
 		</transmission>
 	</xacro:macro>
-	<xacro:Trans Name="right_front_yaw" />
-	<xacro:Trans Name="right_front_hip" />
-	<xacro:Trans Name="right_front_knee" />
+	<xacro:Trans Name="left_front_pitch" />
+	<xacro:Trans Name="left_front_hip" />
+	<xacro:Trans Name="left_front_knee" />
 </robot>

File: qr_description/urdf/single_leg.urdf.xacro (robot description, xacro)
@@ -65,5 +65,5 @@
 			</inertial>
 		</link>
-		<joint name="${Name}_yaw" type="revolute">
+		<joint name="${Name}_pitch" type="revolute">
 			<origin xyz="${X_Dir*(BODY_X/2-SHOD_L/2)} ${Y_Dir*(BODY_Y/2-SHOD_R)} ${-SHOD_R*2}" rpy="0 0 0"/>
 			<parent link="${Parent_Link}"/>
@@ -138,7 +138,7 @@
 	<!--***************************************************************-->
 	<xacro:Body Name="body" Mass="10"/>
-	<xacro:Shoulder Name="right_front"  Mass="1" Parent_Link="body" X_Dir = "1"  Y_Dir = "-1"/>
-	<xacro:LEG Name="right_front"   Mass="1" Limit_Up = "2" Limit_Low="0"/>
-	<xacro:SHINE Name="right_front"  Mass="1" Limit_Up = "0" Limit_Low="-2"/>
+	<xacro:Shoulder Name="left_front"  Mass="1" Parent_Link="body" X_Dir = "1"  Y_Dir = "-1"/>
+	<xacro:LEG Name="left_front"   Mass="1" Limit_Up = "2" Limit_Low="0"/>
+	<xacro:SHINE Name="left_front"  Mass="1" Limit_Up = "0" Limit_Low="-2"/>
 	<link name="world"/>
 	<joint name="base_fixed" type="fixed">

File: qr_description/urdf/single_leg.xacro (robot description, xacro)
@@ -1,6 +1,6 @@
 <?xml version="1.0"?>
 <robot xmlns:xacro="http://www.ros.org/wiki/xacro" name="dragon">
-  <xacro:include filename="$(find qr_description)/urdf/single_leg.urdf.xacro"/>
-  <xacro:include filename="$(find qr_description)/urdf/single_leg.transmission.xacro"/>
-  <xacro:include filename="$(find qr_description)/urdf/single_leg.gazebo.xacro"/>
+  <xacro:include filename="$(find dragon_description)/urdf/single_leg.urdf.xacro"/>
+  <xacro:include filename="$(find dragon_description)/urdf/single_leg.transmission.xacro"/>
+  <xacro:include filename="$(find dragon_description)/urdf/single_leg.gazebo.xacro"/>
 </robot>

Commit message: temp

File: qr_description/urdf/dinasour.urdf.xacro (robot description, xacro)
@@ -9,6 +9,6 @@
 	<xacro:property name="Effort_Limit"  value="50" />
 	<xacro:property name="Velocity_Limit" value="1" />
-	<xacro:property name="BODY_X"        value="0.8" />
-	<xacro:property name="BODY_Y"        value="0.5" />
+	<xacro:property name="BODY_X"        value="0.553" />
+	<xacro:property name="BODY_Y"        value="0.336" />
 	<xacro:property name="BODY_Z"        value="0.1" />
 	<xacro:property name="SHOD_R"        value="0.04" />

Commit message: Test

File: qr_description/urdf/dinasour.urdf.xacro (robot description, xacro)
@@ -133,4 +133,22 @@
 			<limit lower="${Limit_Low}" upper="${ Limit_Up}" effort="${Effort_Limit}" velocity="${Velocity_Limit}"/>
 		</joint>
+		<link name="${Name}_foot">
+			<visual>
+				<origin xyz="0 0 ${-SHE_L/2}" rpy="0 0 0"/>
+				<geometry>
+					<cylinder radius="${SHE_R}" length="0.0001"/>
+				</geometry>
+			</visual>
+			<collision>
+				<origin xyz="0 0 ${-SHE_L/2}" rpy="0 0 0"/>
+				<geometry>
+					<cylinder radius="${SHE_R}" length="0.0001"/>
+				</geometry>
+			</collision>
+		</link>
+		<joint name="${Name}_foot_fixed" type="fixed">
+			<parent link="${Name}_shine"/>
+			<child link="${Name}_foot"/>
+		</joint>
 	</xacro:macro>
 	<!--***************************************************************-->
@@ -150,8 +168,8 @@
 	<xacro:SHINE Name="left_back"   Mass="1" Limit_Up = "2" Limit_Low="-2" />
 	<xacro:SHINE Name="right_back"  Mass="1" Limit_Up = "2" Limit_Low="-2" />
-	<link name="world"/>
+	<!--link name="world"/>
 	<joint name="base_fixed" type="fixed">
 		<parent link="world"/>
 		<child link="body"/>
-	</joint>
+	</joint-->
 </robot>
